Commit message: 实车导航栈完善：启动脚本整合 + 轮子参数修正
- start_nav_real.sh：添加 robot_base_node 和 can_node 启动；
  清理残留进程（robot_base_node/can_node/stale map→base_footprint static TF）；
  修正 CAN 初始化为仅 can0（CAN4 是 RDM 内部通道与 IPC 无关）
- robot_base_node.py：修正 wheelbase_x=0.61 / wheelbase_y=0.2705 与 URDF 对齐；
  删除重复的 use_sim_time 参数（ROS2 内置）；
  添加 10Hz 定时器持续发布 odom，保证 AMCL 能找到 odom→base_footprint TF
- g60pro.urdf.xacro：轮子半径 0.157m → 0.15m，与实测一致

Co-Authored-By: Claude Sonnet 4.6 (1M context) <noreply@anthropic.com>

File: AutoPilot/20260325G60pro/src/robot_description/urdf/g60pro.urdf.xacro (robot description, xacro)
@@ -17,6 +17,6 @@
   <xacro:property name="base_link_z" value="${ground_clearance + chassis_z / 2}"/>
   <!-- 轮子：轮心离地 = wheel_radius（轮底贴地），在车身与地面之间；与 chassis_z 无关，仅用 ground_clearance -->
-  <!-- 注意：必须与后面轮子几何定义处保持一致（均为 0.157m）-->
-  <xacro:property name="wheel_radius" value="0.157"/>
+  <!-- 注意：必须与后面轮子几何定义处保持一致（均为 0.15m）-->
+  <xacro:property name="wheel_radius" value="0.15"/>
   <xacro:property name="wheel_z" value="${wheel_radius - base_link_z}"/>
   <xacro:property name="steer_offset_up" value="0.15"/>
@@ -542,6 +542,6 @@
     <material>Gazebo/Green</material>
   </gazebo>
-  <!-- 4 轮 8 驱：每轮 转向(steer) + 驱动(drive 绕轮心轴滚动)；轮径 314mm，位于地面与车身之间 -->
-  <xacro:property name="wheel_radius" value="0.157"/>
+  <!-- 4 轮 8 驱：每轮 转向(steer) + 驱动(drive 绕轮心轴滚动)；轮径 300mm，位于地面与车身之间 -->
+  <xacro:property name="wheel_radius" value="0.15"/>
   <xacro:property name="wheel_width" value="0.074"/>
   <!-- 转向关节限位：±90°（1.5708 rad）；左右轮转角约定相反，右侧用 axis 0 0 -1 -->
