Commit message: 单线激光雷达的Z坐标，要高于map/costmap，才能在costmap生成膨胀区

File: AutoPilot/20260325G60pro/src/robot_description/urdf/g60pro.urdf.xacro (robot description, xacro)
@@ -26,5 +26,5 @@
   <xacro:property name="camera_z" value="${camera_height_from_ground - base_link_z}"/>
   <!-- 单线雷达离地高度（相对 base_footprint），相对 base_link 的 z -->
-  <xacro:property name="single_lidar_height_from_ground" value="0.486"/>
+  <xacro:property name="single_lidar_height_from_ground" value="1.5"/>
   <xacro:property name="single_lidar_z" value="${single_lidar_height_from_ground - base_link_z}"/>
   <!-- 单线雷达在车身外：前后超出 single_lidar_outset_x，左右超出 single_lidar_outset_y -->
@@ -229,5 +229,5 @@
     <xacro:robosense_16_lidar name="rs16" parent="base_link" xyz="${multi_lidar_offset_x} 0 ${multi_lidar_z}" rpy="0 0 0"/>
   </xacro:unless>
-  <!-- 单线 1: 物理右前（橙色），车身外；倒装(roll 180°) + 315° 扇区朝右前(yaw -45°) -->
+  <!-- 单线 1: 物理右前（橙色），车身外；正装(roll 0°) + 250° 扇区朝右前(yaw -45°) -->
   <link name="single_lidar_1_link">
     <visual>
@@ -240,5 +240,5 @@
     <parent link="base_link"/>
     <child link="single_lidar_1_link"/>
-    <origin xyz="${single_lidar_front_x} ${single_lidar_right_y} ${single_lidar_z}" rpy="3.14159 0 -0.785398"/>
+    <origin xyz="${single_lidar_front_x} ${single_lidar_right_y} ${single_lidar_z}" rpy="0 0 -0.785398"/>
   </joint>
   <!-- 单线 1 仿真：ray 传感器发布 LaserScan，话题 /lidar/single_1/scan，与 hardware_spec 一致 -->
@@ -252,6 +252,6 @@
             <samples>360</samples>
             <resolution>1</resolution>
-            <min_angle>-2.35619</min_angle>
-            <max_angle>2.35619</max_angle>
+            <min_angle>-2.26893</min_angle>
+            <max_angle>2.26893</max_angle>
           </horizontal>
         </scan>
@@ -278,5 +278,5 @@
     </sensor>
   </gazebo>
-  <!-- 单线 2: 物理左后（绿色），车身外；倒装(roll 180°) + 225° 扇区朝左后(yaw 135°) -->
+  <!-- 单线 2: 物理左后（绿色），车身外；正装(roll 0°) + 250° 扇区朝左后(yaw 135°) -->
   <link name="single_lidar_2_link">
     <visual>
@@ -289,5 +289,5 @@
     <parent link="base_link"/>
     <child link="single_lidar_2_link"/>
-    <origin xyz="${single_lidar_rear_x} ${single_lidar_left_y} ${single_lidar_z}" rpy="3.14159 0 2.35619"/>
+    <origin xyz="${single_lidar_rear_x} ${single_lidar_left_y} ${single_lidar_z}" rpy="0 0 2.35619"/>
   </joint>
   <!-- 单线 2 仿真：ray 传感器发布 LaserScan，话题 /lidar/single_2/scan，与 hardware_spec 一致 -->
@@ -301,6 +301,6 @@
             <samples>360</samples>
             <resolution>1</resolution>
-            <min_angle>-2.35619</min_angle>
-            <max_angle>2.35619</max_angle>
+            <min_angle>-2.26893</min_angle>
+            <max_angle>2.26893</max_angle>
           </horizontal>
         </scan>
@@ -634,9 +634,9 @@
       <publish_rate>50</publish_rate>
       <!-- 是否发布 /odom 话题 -->
-      <!-- true: 发布 nav_msgs/Odometry 消息 -->
-      <publish_odom>true</publish_odom>
+      <!-- false: 不发布 odom 话题，让 Cartographer 完全接管定位 -->
+      <publish_odom>false</publish_odom>
       <!-- 是否发布 TF 变换 -->
-      <!-- true: 发布 odom -> base_footprint 的动态变换 -->
-      <publish_tf>true</publish_tf>
+      <!-- false: 不发布 odom→base_footprint TF，让 Cartographer 发布 map→base_footprint -->
+      <publish_tf>false</publish_tf>
       <!-- odom 坐标系名称 -->
       <!-- TF 中 frame_id 将是 "odom" -->

Commit message: fix: 单线雷达高度修正为 0.486m + 新增仿真纯定位模式 + 地图 v9/v10
- URDF: single_lidar_height_from_ground 1.5m → 0.486m
- 新增仿真 Cartographer 纯定位模式（cartographer_sim_localization.lua +
  slam_sim_localization.launch.py）
- 新增 start_nav_sim_map.sh 脚本，支持加载已有地图进行仿真导航
- RViz: 移除 odom frame，TF 树对齐实车设计（map→base_footprint）
- 保存地图 g60pro_v9 / g60pro_v10

File: AutoPilot/20260325G60pro/src/robot_description/urdf/g60pro.urdf.xacro (robot description, xacro)
@@ -26,5 +26,5 @@
   <xacro:property name="camera_z" value="${camera_height_from_ground - base_link_z}"/>
   <!-- 单线雷达离地高度（相对 base_footprint），相对 base_link 的 z -->
-  <xacro:property name="single_lidar_height_from_ground" value="1.5"/>
+  <xacro:property name="single_lidar_height_from_ground" value="0.486"/>
   <xacro:property name="single_lidar_z" value="${single_lidar_height_from_ground - base_link_z}"/>
   <!-- 单线雷达在车身外：前后超出 single_lidar_outset_x，左右超出 single_lidar_outset_y -->
